File: nrf54_board/nrf54_boards.kicad_pcb (KiCad board)
At the start: 2 copper layers, 22 parts, among them U1 nRF54L15-QFAA, X1 32.768kHz, X2 32MHz

Commit message: update
Parts:
- added J1: Conn_01x04_Pin, Connector_PinHeader_2.54mm:PinHeader_1x04_P2.54mm_Vertical, F.Cu at (127.5, 96.0)

Commit message: update
Parts:
- moved C8 0.50 mm to (122.0, 90.5)
Routing:
- net GND: track 0.00 -> 79.2 mm, vias 0 -> 6
- net VDD_nRF: track 0.00 -> 54.8 mm, vias 0 -> 1
- net /DECA: track 0.00 -> 24.0 mm, vias 0 -> 2
- net /SWDCLK: track 0.00 -> 9.93 mm, vias 0 -> 1
- net /SWDIO: track 0.00 -> 9.89 mm
- net /DECD: track 0.00 -> 8.21 mm
- net /XC1: track 0.00 -> 6.27 mm
- net /DCC: track 0.00 -> 5.34 mm
- net Net-(U1A-~{RESET}): track 0.00 -> 4.46 mm
- net /P1.00/XL1: track 0.00 -> 3.90 mm
- net /P1.01/XL2: track 0.00 -> 3.85 mm
- net Net-(C9-Pad2): track 0.00 -> 2.26 mm
- net Net-(U1A-ANT): track 0.00 -> 2.24 mm
- net Net-(C6-Pad2): track 0.00 -> 2.19 mm
- net /RF: track 0.00 -> 1.96 mm
Other:
- board outline added: 34.5 x 31.5 mm

Commit message: update
Other:
- board size 34.5 x 31.5 mm -> 34.5 x 26 mm
Changed lines of the file:
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@@
 	)
 	(gr_rect
-		(start 105 71)
-		(end 139.5 102.5)
+		(start 105 73.5)
+		(end 139.5 99.5)
 		(stroke
 			(width 0.05)
