File: nrf54_board/nrf54_boards.kicad_sch (KiCad schematic)
At the start: 22 parts, among them U1 ${ALTIUM_VALUE}, X1 ${ALTIUM_VALUE}, X2 ${ALTIUM_VALUE}

Commit message: update
Parts:
- added J1: Conn_01x04_Pin, Connector_PinHeader_2.54mm:PinHeader_1x04_P2.54mm_Vertical, symbol Connector:Conn_01x04_Pin
Connections:
- net GND: now also J1.3 (Pin_3)
- net SWDCLK: now also J1.2 (Pin_2)
- net SWDIO: now also J1.1 (Pin_1)
- net VDD_nRF: now also J1.4 (Pin_4)

Commit message: update
Parts:
- added J2: UART Connector, symbol Connector:Conn_01x06_Pin
- J1: value Conn_01x04_Pin -> SWD Connector
Changed lines of the file:
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@@
 			"QQBBAEEAQQBBAEEAQQBBAEEAQQBBAEEAQQBBAEEAQQBBAEEAQQBBAEEAQQBBAEEAQQBBAEEAQQBB"
 			"AEEAQQBBAEEAQQBBAEEAQQBBAEEAQQBBAEEAQQBBAEEAQQBBAEEAQQBBAEEAQQBBAEEAQQBBAEEA"
+			"QQBBAEEAQQBBAEEAQQBBAEEAQQBBAEEAQQBBAEEAQQBBAEEAQQBEAEEAdwBNAHAANgBlAG4ALwBm"
+			"ADMAOQAvAC8ALwAvAC8ALwAvAC8ALwAvAC8ALwAvAC8ALwAvAC8ALwAvAC8ALwAvAC8ALwAvAC8A"
+			"LwAvAC8ALwAvAC8ALwAvAC8ALwAvAC8ALwAvAC8ALwAvAC8ALwAvAC8ALwAvAC8ALwAvAC8ALwAv"
+			"AC8ALwAvAC8ALwAvAC8ALwAvAC8ALwAvAC8ALwAvAC8ALwAvAC8ALwAvAFIAVQBWAEYAQQBBAEEA"
+			"QQBBAEEAQQBBAEEAQQBBAEEAQQBBAEEAQQBBAEEAQQBBAEEAQQBBAEEAQQBBAEEAQQBBAEEAQQBB"
+			"AEEAQQBBAEEAUQBFAEIAQQA3AGUAMwB0AC8ALwAvAC8ALwAvAC8ALwAvAC8ALwAvAC8ALwAvAC8A"
+			"LwAvAC8ALwAvAC8ALwAvAC8ALwAvAC8ALwAvAC8ALwAvAC8ALwAvAC8ALwAvAC8ALwAvAC8ALwAv"
+			"AC8ALwAvAC8ALwAvAC8ALwAvAC8ALwBnAG8ASwBDAEEAQQBBAEEAQQBBAEEAQQBBAEEAQQBBAEEA"
+			"QQBBAEEAQQBBAEEAQQBBAEEAQQBBAEoAUwBVAGwANgArAHYAcgAvAC8ALwAvAC8ALwAvAC8ALwAv"
+			"AC8ALwAvAC8ALwAvAC8ALwAvAC8ALwAvAC8ALwAvAC8ALwAvAC8ALwAvAC8ALwAvAC8ALwAvAC8A"
+			"LwAvAC8ALwAvAC8ALwAvAC8ALwAvAC8ALwAvAC8ALwAvAC8ALwAvAC8ALwAvAC8ALwAvAHkAOAB2"
+			"AEwARAB3ADgAUABBAEEAQQBBAEEAQQBBAEEAQQBBAEEAQQBBAEEAQQBBAEEAQQBBAEEAQQBBAEEA"
+			"QQBBAEEAQQBBAEEAQQBBAEEAQQBBAEEAQQBBAEEAQQBBAEEAQQBBAEEAQQBBAEEAQQBBAEEAQQBB"
+			"AEEAQQBBAEEAQQBBAEEAQQBBAEEAQQBBAEEAQQBBAEEAQQBBAEEAQQBBAEEAQQBBAEEAQQBBAEEA"
+			"QQBBAEEAQQBBAEEAQQBBAEEAQQBBAEEAQQBBAEEAQQBBAEEAQQBBAEMAUQBrAEoAZQBIAGgANAAr"
+			"AGYAbgA1AC8ALwAvAC8ALwAvAC8ALwAvAC8ALwAvAC8ALwAvAC8ALwAvAC8ALwAvAC8ALwAvAC8A"
+			"LwAvAC8ALwAvAC8ALwAvAC8ALwAvAC8ALwAvAC8ALwAvAC8ALwAvAC8ALwAvAC8ALwAvAC8ALwAv"
+			"AC8ALwAvAC8ALwAvAC8ALwAvAC8ALwAvAC8ALwAvAC8ALwAvAC8ALwAvAC8AbgA1ACsAZgBBAEEA"
 			"QQBBAEEAQQBBAEEAQQBBAEEAQQBBAEEAQQBBAEEAQQBBAEEAQQ=="
 		)
@@
 			"awAwAFgASABrADAAWABIAGsAMABYAEgAawAwAFgASABrADAAWABIAGsAMABYAEgAawAwAFgASABr"
 			"ADAAWABIAGsAMABYAEgAawAwAFgASABrADAAWABIAGsAMABYAEgAawAwAFgASABrADAAWABIAGsA"
-			"MABYAEgAawAwAFgASABrAA=="
+			"MABYAEgAawAwAFgASABrADAAWABIAGsAMABYAEgAawAwAFgASABrADAAWABIAGsAMABYAEgAawAw"
+			"AFgASABrADAAWABIAGsAMABYAEgAawAwAFgASABrADAAWABIAGsAMABYAEgAawAwAFgASABrADAA"
+			"WABIAGsAMABYAEgAawAwAFgASABrADAAWABIAGsAMABYAEgAawAwAFgASABrADAAWABIAGsAMABY"
+			"AEgAawAwAFgASABrADAAWABIAGsAMABYAEgAawAwAFgASABrADAAWABIAGsAMABYAEgAawAwAFgA"
+			"SABrADAAWABIAGsAMABYAEgAawAwAFgASABrADAAWABIAGsAMABYAEgAawAwAFgASABrADAAWABI"
+			"AGsAMABYAEgAawAwAFgASABrADAAWABIAGsAMABYAEgAawAwAFgASABrADAAWABIAGsAMABYAEgA"
+			"awAwAFgASABrADAAWABIAGsAMABYAEgAawAwAFgASABrADAAWABIAGsAMABYAEgAawAwAFgASABr"
+			"ADAAWABIAGsAMABYAEgAawAwAFgASABrADAAWABIAGsAMABYAEgAawAwAFgASABrADAAWABIAGsA"
+			"MABYAEgAawAwAFgASABrADAAWABIAGsAMABYAEgAawAwAFgASABrADAAWABIAGsAMABYAEgAawAw"
+			"AFgASABrADAAWABIAGsAMABYAEgAawAwAFgASABrADAAWABIAGsAMABYAEgAawAwAFgASABrADAA"
+			"WABIAGsAMABYAEgAawAwAFgASABrADAAWABIAGsAMABYAEgAawAwAFgASABrADAAWABIAGsAMABY"
+			"AEgAawAwAFgASABrADAAWABIAGsAMABYAEgAawAwAFgASABrADAAWABIAGcAeQBsAHoAVgB0AEIA"
+			"egBRAHEAZwBEAFEAcQBnAEQAUQBxAGcARABRAHEAZwBEAFEAcQBnAEQAUQBxAGcARABRAHEAZwBE"
+			"AFEAcQBnAEQAUQBxAGcARABRAHEAZwBEAFEAcQBnAEQAUQBxAGcARABRAHEAZwBEAFEAcQBnAEQA"
+			"UQBxAGcARABRAHEAZwBEAFEAcQBnAEQAUQBxAGcARABRAHEAZwBEAFEAcQBnAEQAUQBxAGcARABR"
+			"AHEAZwBEAFEAcQBnAEQAUQBxAGcARABRAHEAZwBEAFEAcQBnAEQAUQBxAGcARABRAHEAZwBEAFEA"
+			"cQBnAEQAUQBxAGcARABRAHEAZwBEAFEAcQBnAEQAUQBxAGcARABRAHEAZwBEAFEAcQBnAEQAUQBx"
+			"AGcARABRAHEAZwBEAFEAcQBnAEQAUQBxAGcARABRAHEAZwBEAFEAcQBnAEQAUQBxAGcARABRAHEA"
+			"ZwBEAFEAcQBnAEQAUQBxAA=="
 		)
 	)
@@
 			)
 		)
-		(property "Value" "Conn_01x04_Pin"
+		(property "Value" "SWD Connector"
 			(at 103.505 152.4 0)
 			(effects
@@
 					(unit 1)
 				)
+			)
+		)
+	)
+	(symbol
+		(lib_id "Connector:Conn_01x06_Pin")
+		(at 203.2 109.22 0)
+		(unit 1)
+		(exclude_from_sim no)
+		(in_bom yes)
+		(on_board yes)
+		(dnp no)
+		(fields_autoplaced yes)
+		(property "Reference" "J2"
+			(at 203.835 99.06 0)
+			(effects
+				(font
+					(size 1.27 1.27)
+				)
+			)
+		)
+		(property "Value" "UART Connector"
+			(at 203.835 101.6 0)
+			(effects
+				(font
+					(size 1.27 1.27)
+				)
+			)
+		)
+		(property "Footprint" ""
+			(at 203.2 109.22 0)
+			(effects
+				(font
+					(size 1.27 1.27)
+				)
+				(hide yes)
+			)
+		)
+		(property "Datasheet" "~"
+			(at 203.2 109.22 0)
+			(effects
+				(font
+					(size 1.27 1.27)
+				)
+				(hide yes)
+			)
+		)
+		(property "Description" "Generic connector, single row, 01x06, script generated"
+			(at 203.2 109.22 0)
+			(effects
+				(font
+					(size 1.27 1.27)
+				)
+				(hide yes)
+			)
+		)
+		(pin "4"
+		)
+		(pin "5"
+		)
+		(pin "1"
+		)
+		(pin "3"
+		)
+		(pin "6"
+		)
+		(pin "2"
+		)
+		(instances
+			(project ""
+				(path "/fde990c2-10fb-45a6-b818-f82379edb904"
+					(reference "J2")
+					(unit 1)
+				)
